File: BBBLedHW.kicad_sch (KiCad schematic)
At the start: 40 parts, among them J3 Barrel_Jack_Switch, Q1 2N7002, U1 STM32WB55CEUx, U2 TPS7A2033DBV, U3 SN74LVC1T45DBV, U4 ADP2303ARDZ-5.0, X1 32MHz, X2 32kHz768

Commit message: Final touches before review
Parts:
- added C19: 100n, symbol Device:C
- added C20, C21: 100u, symbol Device:C
- added C22: 47u, symbol Device:C
- added D2: LED_GREEN, symbol Device:LED
- added D3: LED_RED, symbol Device:LED
- added D4: SSB43L 4A 30V, symbol Device:D_Schottky
- added J1: USB_B, symbol Connector:USB_B
- added R10: 220R, symbol Device:R
- added R7, R8: 680R, symbol Device:R
- added R9: 5k1, symbol Device:R
- added SW1: SW_Push, symbol Switch:SW_Push
- added U5: USBLC6-2SC6, Package_TO_SOT_SMD:SOT-23-6, symbol Power_Protection:USBLC6-2SC6
- ANT1: value ~ -> PCB Trace Antenna
- C15: renamed from C14; value C -> 10p
- C16: renamed from C15; value C -> 10p
- C18: renamed from C13; value 1u -> 10u
- J2: value ~ -> WS2812 3x1 Header
- J4: renamed from J1; value ~ -> Molex 2.54 2-rows 10-pins
- renumbered C4 to C1, C18 to C10, C10 to C11, C11 to C12, C12 to C13, C9 to C14, C8 to C17, C3 to C2, C2 to C3, C1 to C4, C17 to C8, C16 to C9, D2 to D1, L2 to L1, L3 to L2, L1 to L3, R4 to R2, R5 to R3, R2 to R4, R3 to R5, U3 to U1, U4 to U2, U1 to U3, U2 to U4
Connections:
- net LED_LLC is gone; now on net LED_DATA: U1.3 (A)
- net +3V3: now also SW1.2
- net +5V: now also J2.3 (5V), C20.1, C21.1, C22.1, D4.1 (K), U5.5 (VBUS)
- net GND: now also U1.5 (DIR), C19.2, C20.2, C21.2, C22.2, D2.1 (K), D3.1 (K), J1.4 (GND), J1.5 (Shield), R9.2, U5.2 (GND)
- net LED_DATA: no longer U1.4 (B)
- net VBUS: no longer J2.3 (5V)
- net MCU_LSE_OUT: now reaches C16.1, U3.3 (PC15), X2.2
- net MCU_LED_GREEN: now reaches U3.13 (PA4)
- net MCU_LED_GREEN: now also R7.1
- net MCU_LED_RED: now reaches U3.14 (PA5)
- net MCU_LED_RED: now also R8.1
- net MCU_LSE_IN: now reaches C15.1, U3.2 (PC14), X2.1
- net MCU_RF: now reaches C8.1, L1.2, U3.21 (RF1)
- net MCU_HSE_OUT: now reaches U3.24 (OSC_OUT), X1.1
- net MCU_HSE_IN: now reaches U3.25 (OSC_IN), X1.3
- net USB_D-: now reaches U3.37 (PA11)
- net USB_D-: now also U5.4 (I/O2)
- net USB_D+: now reaches U3.38 (PA12)
- net USB_D+: now also U5.6 (I/O1)
- net MCU_BOOT0: now reaches U3.4 (PH3)
- net MCU_BOOT0: now also C19.1, R10.1, R9.1
- net MCU_LLC: now reaches U3.9 (PA0)
- net MCU_LLC: now also U1.4 (B)
- net MICROSTRIP: now reaches FL1.3, L2.1
- net RF_ANT: now reaches ANT1., C10.1, L2.2
- net 5V_EN renamed REG_EN
- net RF_LPF: no longer names the net of C9.1, FL1.1, L1.1
- net SWD_O: no longer names the net of U3.43 (PB3)
- net USB_5V renamed USB_EN
- net USB_EN: now also D4.2 (A), J1.1 (VBUS)
- new net: D2.2 (A), R7.2
- new net: J1.3 (D+), U5.1 (I/O1)
- new net: J1.2 (D-), U5.3 (I/O2)
- new net: D3.2 (A), R8.2
- new net: R10.2, SW1.1
- no-connect marks 6 -> 30
Other:
- note added: "1.0"
- note added: "24/07/25"
- note added: "3V3 Regulator"
- note added: "5V Regulator Disable"
- note added: "BLE Board for LED Light Strip"
- note added: "Debug Perhiperals"
- note added: "H&LSE Oscillators"
- note added: "MCU"
- note added: "Mitchell Mesman"
- note added: "Power Connectors"
- note added: "RF Matching Networks and Antenna"
- note removed: "3V3 MCU"
- note removed: "Buck Disable"
- note removed: "Power"
- note removed: "RF Matching Networks"
- moved on the sheet: C1, C10, C11, C12, C13, C14, C15, C16, C17, C18, C2, C3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

Commit message: Add reviewed schematic
Connections:
- net +5V: no longer U5.5 (VBUS)
- net USB_EN: now also U5.5 (VBUS)
Other:
- moved on the sheet: C10, C8, C9, D4

Commit message: Final touches before assigning footprints
Parts:
- added C23, C24, C26, C27: 100n, symbol Device:C
- added C25, C28: 10n, symbol Device:C
- added D5: LED_RED, symbol Device:LED
- added Q3: 2N7002, Package_TO_SOT_SMD:SOT-23, symbol Transistor_FET:2N7002
- added R11: 1k, symbol Device:R
- ANT1: footprint (none) -> bbbled:TraceAntenna
- C11: value 10u 25V -> 47u 25V
- D2: value LED_GREEN -> LED_RED
- FL1: footprint LFB182G45CGFD436:FIL_LFB182G45CGFD436 -> bbbled:FIL_LFB182G45CGFD436
- R7, R8: value 680R -> 1k
Connections:
- net +3V3: now also R7.1, R8.1, C24.1
- net +5V: now also C23.1, C27.1, C28.1, R11.1
- net GND: now also C23.2, C24.2, C25.2, C26.2, C27.2, C28.2, Q3.2 (S); no longer D2.1 (K), D3.1 (K)
- net VBUS: now also C25.1, C26.1
- net at R1.1, U2.4 (PGOOD): now also Q3.1 (G)
- net at R7.2: now also D3.2 (A); no longer D2.2 (A)
- net at R8.2: now also D2.2 (A); no longer D3.2 (A)
- net MCU_LED_GREEN renamed MCU_LED_1
- net MCU_LED_1: now also D2.1 (K); no longer R7.1
- net MCU_LED_RED renamed MCU_LED_2
- net MCU_LED_2: now also D3.1 (K); no longer R8.1
- new net: D5.2 (A), R11.2
- new net: D5.1 (K), Q3.3 (D)
Other:
- moved on the sheet: C11, C12, C13, C15, C16, C17, C18, C22, D1, D2, D3, L3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

Commit message: Chosen components, footprints, 3d models and PCB constraints. Next step - placing and routing!
Parts:
- added C29: 100p, Capacitor_SMD:C_0402_1005Metric, symbol Device:C
- added Q2, Q4: 2N7002, Package_TO_SOT_SMD:SOT-23, symbol Simulation_SPICE:NMOS
- added R12, R13: 10k, Resistor_SMD:R_0402_1005Metric, symbol Device:R
- C1, C12, C14, C19, C2, C23, C24, C26, C27, C3, C4, C5, C6, C7: footprint (none) -> Capacitor_SMD:C_0402_1005Metric; Distributor Link (none) -> https://www.digikey.co.nz/en/products/detail/kyocera-avx/KG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; MANUFACTURER (none) -> KYOCERA AVX; Manufacturer Part Number (none) -> KGM05AR71E104KH; Price (none) -> 0.14
- C10: footprint (none) -> Capacitor_SMD:C_0402_1005Metric; Distributor Link (none) -> https://www.digikey.co.nz/en/products/detail/murata-electro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; MANUFACTURER (none) -> Murata Electronics; Manufacturer Part Number (none) -> GRM1555C1H1R2WA01D; Price (none) -> 0.2
- C11: value 47u 25V -> 10u; footprint (none) -> Capacitor_SMD:C_0805_2012Metric; Distributor Link (none) -> https://www.digikey.co.nz/en/products/detail/murata-electro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; MANUFACTURER (none) -> Murata Electronics; Manufacturer Part Number (none) -> GRM21BR61E106KA73K; Price (none) -> 0.29
- C13, C22: value 47u -> 47u 6.3V; footprint (none) -> Capacitor_SMD:C_0805_2012Metric; Distributor Link (none) -> https://www.digikey.co.nz/en/products/detail/tdk-corporatio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; MANUFACTURER (none) -> TDK Corporation; Manufacturer Part Number (none) -> C2012X5R0J476M125AC; Price (none) -> 1.04
- C15, C16: footprint (none) -> Capacitor_SMD:C_0402_1005Metric; Distributor Link (none) -> https://www.digikey.co.nz/en/products/detail/kyocera-avx/KG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; MANUFACTURER (none) -> KYOCERA AVX; Manufacturer Part Number (none) -> KGM05ACG1H100JN; Price (none) -> 0.18
- C17: footprint (none) -> Capacitor_SMD:C_0402_1005Metric; Distributor Link (none) -> https://www.digikey.co.nz/en/products/detail/murata-electro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; MANUFACTURER (none) -> Murata Electronics; Manufacturer Part Number (none) -> GRT155R70J105KE01D; Price (none) -> 0.18
- C18: footprint (none) -> Capacitor_SMD:C_0805_2012Metric; Distributor Link (none) -> https://www.digikey.co.nz/en/products/detail/murata-electro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; MANUFACTURER (none) -> Murata Electronics; Manufacturer Part Number (none) -> GRM21BR61E106KA73K; Price (none) -> 0.29
- C20, C21: footprint (none) -> bbbled:WCAP-ASLI_5X5.5_DXL_; Distributor Link (none) -> https://www.digikey.co.nz/en/products/detail/w%C3%BCrth-ele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; MANUFACTURER (none) -> Würth Elektronik; Manufacturer Part Number (none) -> 865080142007; Price (none) -> 0.38
- C25, C28: footprint (none) -> Capacitor_SMD:C_0402_1005Metric; Distributor Link (none) -> https://www.digikey.co.nz/en/products/detail/yageo/CC0402KR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; MANUFACTURER (none) -> YAGEO; Manufacturer Part Number (none) -> CC0402KRX7R8BB103; Price (none) -> 0.18
- C8: footprint (none) -> Capacitor_SMD:C_0402_1005Metric; Distributor Link (none) -> https://www.digikey.co.nz/en/products/detail/murata-electro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; MANUFACTURER (none) -> Murata Electronics; Manufacturer Part Number (none) -> GRM1555C1HR30WA01D; Price (none) -> 0.29
- C9: footprint (none) -> Capacitor_SMD:C_0402_1005Metric; Distributor Link (none) -> https://www.digikey.co.nz/en/products/detail/murata-electro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; MANUFACTURER (none) -> Murata Electronics; Manufacturer Part Number (none) -> GRM1555C1HR80BA01D; Price (none) -> 0.2
- D1, D4: footprint (none) -> bbbled:DIODE_DO214AA_MBRS-L; Distributor Link (none) -> https://www.digikey.co.nz/en/products/detail/vishay-general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; MANUFACTURER (none) -> Vishay General Semiconductor - Diodes Division; Manufacturer Part Number (none) -> SSB43L-E3/52T; Price (none) -> 0.7
- D2, D3, D5: footprint (none) -> LED_SMD:LED_0603_1608Metric; Distributor Link (none) -> https://www.digikey.com/en/products/detail/liteon/LTST-C190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; MANUFACTURER (none) -> Lite-On Inc.; Manufacturer Part Number (none) -> LTST-C190KRKT; Price (none) -> 0.14
- FL1: Distributor Link (none) -> https://www.digikey.co.nz/en/products/detail/murata-electro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; Manufacturer Part Number (none) -> LFB182G45CGFD436; Price (none) -> 0.36
- J1: footprint (none) -> bbbled:CONN_10118194-0001LF_AMP; Distributor Link (none) -> https://www.digikey.co.nz/en/products/detail/amphenol-cs-fc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; MANUFACTURER (none) -> Amphenol ICC (FCI); Manufacturer Part Number (none) -> 10118194-0001LF; Price (none) -> 0.77
- J3: footprint (none) -> bbbled:TENSILITY_54-00131; Distributor Link (none) -> https://www.digikey.com/en/products/detail/tensility-intern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; MANUFACTURER (none) -> Tensility International Corp; Manufacturer Part Number (none) -> 54-00131; Price (none) -> 0.82
- J4: footprint (none) -> bbbled:CONN10_302-S101_OST; Distributor Link (none) -> https://www.digikey.co.nz/en/products/detail/on-shore-techn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; MANUFACTURER (none) -> On Shore Technology Inc.; Manufacturer Part Number (none) -> 302-S101; Price (none) -> 0.47
- L1: footprint (none) -> Inductor_SMD:L_0402_1005Metric; Distributor Link (none) -> https://www.digikey.co.nz/en/products/detail/murata-electro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; MANUFACTURER (none) -> Murata Electronics; Manufacturer Part Number (none) -> LQG15HS2N7S02D; Price (none) -> 0.18
- L2: footprint (none) -> Inductor_SMD:L_0402_1005Metric; Distributor Link (none) -> https://www.digikey.co.nz/en/products/detail/murata-electro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; MANUFACTURER (none) -> Murata Electronics; Manufacturer Part Number (none) -> LQG15HS3N6S02D; Price (none) -> 0.18
- L3: footprint (none) -> bbbled:IND_CLF10060NIT-4R7N-D; Distributor Link (none) -> https://www.digikey.co.nz/en/products/detail/tdk-corporatio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; MANUFACTURER (none) -> TDK Corporation; Manufacturer Part Number (none) -> CLF10060NIT-4R7N-D; Price (none) -> 2.16
- Q1: footprint (none) -> Package_TO_SOT_SMD:SOT-23; Distributor Link (none) -> https://www.digikey.co.nz/en/products/detail/onsemi/2n7002/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; MANUFACTURER (none) -> onsemi; Manufacturer Part Number (none) -> 2N7002; Price (none) -> 0.83
- Q3: Distributor Link (none) -> https://www.digikey.co.nz/en/products/detail/onsemi/2n7002/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; MANUFACTURER (none) -> onsemi; Manufacturer Part Number (none) -> 2N7002; Price (none) -> 0.83
- R1, R4: footprint (none) -> Resistor_SMD:R_0402_1005Metric; Distributor Link (none) -> https://www.digikey.co.nz/en/products/detail/panasonic-elec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; MANUFACTURER (none) -> Panasonic Electronic Components; Manufacturer Part Number (none) -> ERA-2AEB104X; Price (none) -> 0.18
- R10: footprint (none) -> Resistor_SMD:R_0402_1005Metric; Distributor Link (none) -> https://www.digikey.co.nz/en/products/detail/delta-electron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; MANUFACTURER (none) -> Delta Electronics/Cyntec; Manufacturer Part Number (none) -> PFR05S-221-FNH; Price (none) -> 0.18
- R11: value 1k -> 330; footprint (none) -> Resistor_SMD:R_0402_1005Metric; Distributor Link (none) -> https://www.digikey.co.nz/en/products/detail/yageo/RC0402FR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; MANUFACTURER (none) -> YAGEO; Manufacturer Part Number (none) -> RC0402FR-13330RL; Price (none) -> 0.18
- R2: footprint (none) -> Resistor_SMD:R_0402_1005Metric; Distributor Link (none) -> https://www.digikey.co.nz/en/products/detail/yageo/RC0402FR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; MANUFACTURER (none) -> YAGEO; Manufacturer Part Number (none) -> RC0402FR-0768KL; Price (none) -> 0.18
- R3: footprint (none) -> Resistor_SMD:R_0402_1005Metric; Distributor Link (none) -> https://www.digikey.co.nz/en/products/detail/yageo/RC0402FR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; MANUFACTURER (none) -> YAGEO; Manufacturer Part Number (none) -> RC0402FR-0713KL; Price (none) -> 0.18
- R5: footprint (none) -> Resistor_SMD:R_0402_1005Metric; Distributor Link (none) -> https://www.digikey.co.nz/en/products/detail/yageo/RC0402FR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; MANUFACTURER (none) -> YAGEO; Manufacturer Part Number (none) -> RC0402FR-1333KL; Price (none) -> 0.18
- R6: footprint (none) -> Resistor_SMD:R_0402_1005Metric; Distributor Link (none) -> https://www.digikey.co.nz/en/products/detail/yageo/RC0402JR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; MANUFACTURER (none) -> YAGEO; Manufacturer Part Number (none) -> RC0402JR-0710KL; Price (none) -> 0.18
- R7, R8: value 1k -> 160; footprint (none) -> Resistor_SMD:R_0402_1005Metric; Distributor Link (none) -> https://www.digikey.co.nz/en/products/detail/panasonic-elec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; MANUFACTURER (none) -> Panasonic Electronic Components; Manufacturer Part Number (none) -> ERJ-2RKF1600X; Price (none) -> 0.18
- R9: footprint (none) -> Resistor_SMD:R_0402_1005Metric; Distributor Link (none) -> https://www.digikey.co.nz/en/products/detail/yageo/RC0402FR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; MANUFACTURER (none) -> YAGEO; Manufacturer Part Number (none) -> RC0402FR-075K1L; Price (none) -> 0.18
- SW1: footprint (none) -> Button_Switch_SMD:SW_Push_1P1T_NO_CK_KMR2; Distributor Link (none) -> https://www.digikey.co.nz/en/products/detail/c-k/KMR231G-LF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; MANUFACTURER (none) -> C&K; Manufacturer Part Number (none) -> KMR231G LFS; Price (none) -> 1.06
- U1: Distributor Link (none) -> https://www.digikey.co.nz/en/products/detail/texas-instrume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; MANUFACTURER (none) -> Texas Instruments; Manufacturer Part Number (none) -> SN74LVC1T45DBVR; Price (none) -> 0.83
- U2: Distributor Link (none) -> https://www.mouser.com/ProductDetail/Analog-Devices/ADP2303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; MANUFACTURER (none) -> Analog Devices; Manufacturer Part Number (none) -> ADP2303ARDZ-5.0-R7; Price (none) -> 5
- U3: Distributor Link (none) -> https://www.digikey.co.nz/en/products/detail/stmicroelectro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; MANUFACTURER (none) -> STMicroelectronics; Manufacturer Part Number (none) -> STM32WB55CEU6; Price (none) -> 11.68
- U4: Distributor Link (none) -> https://www.digikey.co.nz/en/products/detail/texas-instrume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; MANUFACTURER (none) -> Texas Instruments; Manufacturer Part Number (none) -> TPS7A2433DBVR; Price (none) -> 1.04
- U5: Distributor Link (none) -> https://www.digikey.co.nz/en/products/detail/umw/usblc6-2sc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; MANUFACTURER (none) -> UMW; Manufacturer Part Number (none) -> USBLC6-2SC6; Price (none) -> 1.51
- X1: footprint (none) -> Crystal:Crystal_SMD_2016-4Pin_2.0x1.6mm; Distributor Link (none) -> https://www.digikey.com/en/products/detail/ecs-inc/ECS-320-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; MANUFACTURER (none) -> ECS Inc.; Manufacturer Part Number (none) -> ECS-320-8-37CKM; Price (none) -> 0.89
- X2: footprint (none) -> bbbled:XTAL_NX2012SA_NDK; Distributor Link (none) -> https://www.digikey.com/en/products/detail/ndk-nihon-dempa-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; MANUFACTURER (none) -> NDK (NIHON DEMPA KOGYO CO., LTD); Manufacturer Part Number (none) -> STDMUB1-32.768K; Price (none) -> 0.82
Connections:
- net +3V3: now also R7.2, R8.2, C29.1; no longer R7.1, R8.1
- net GND: now also C29.2, Q2.3 (S), Q4.3 (S), R12.1, R13.1
- net MCU_LED_1: now also Q2.2 (G), R12.2; no longer D2.1 (K)
- net MCU_LED_2: now also Q4.2 (G), R13.2; no longer D3.1 (K)
- net at D3.2 (A): now also R7.1; no longer R7.2
- net at D2.2 (A): now also R8.1; no longer R8.2
- new net: D2.1 (K), Q4.1 (D)
- new net: D3.1 (K), Q2.1 (D)
Other:
- moved on the sheet: C19, D2, D3, R10, R7, R8, R9, SW1
